Commit message: add white wheel

File: src/robot_gazebo/urdf/robot.gazebo.xacro (robot description, xacro)
@@ -109,5 +109,5 @@
     <!-- Front Left Wheel -->
     <gazebo reference="wheel_left_front">
-        <material>Gazebo/Black</material>
+        <material>Gazebo/White</material>
         <surface>
             <friction>
@@ -123,5 +123,5 @@
     <!-- Front Right Wheel -->
     <gazebo reference="wheel_right_front">
-        <material>Gazebo/Black</material>
+        <material>Gazebo/White</material>
         <surface>
             <friction>
@@ -137,5 +137,5 @@
     <!-- Back Left Wheel - Now also a drive wheel -->
     <gazebo reference="wheel_left_back">
-        <material>Gazebo/Black</material>
+        <material>Gazebo/White</material>
         <surface>
             <friction>
@@ -151,5 +151,5 @@
     <!-- Back Right Wheel - Now also a drive wheel -->
     <gazebo reference="wheel_right_back">
-        <material>Gazebo/Black</material>
+        <material>Gazebo/White</material>
         <surface>
             <friction>

Commit message: save deploy

File: src/robot_gazebo/urdf/robot.gazebo.xacro (robot description, xacro)
@@ -105,4 +105,21 @@
         </sensor>
     </gazebo>
+    <!-- Contact sensor for the robot body -->
+    <gazebo reference="base_link">
+        <sensor name="contact_sensor_body" type="contact">
+            <always_on>true</always_on>
+            <update_rate>100</update_rate>
+            <contact>
+                <collision>base_link_collision</collision>
+            </contact>
+            <plugin name="gazebo_ros_bumper_body" filename="libgazebo_ros_bumper.so">
+                <ros>
+                    <namespace>/robot</namespace>
+                    <remapping>bumper_states:=cfg/touched</remapping>
+                </ros>
+                <frame_name>base_link</frame_name>
+            </plugin>
+        </sensor>
+    </gazebo>
     <!-- Note: Wheel-ground collisions will be filtered in software by checking collision names -->
     <!-- WHEEL FRICTION SETTINGS FOR 4WD SYSTEM -->
